Commit message: Make URDF links first-class parts and convert assemblies between URDF and ASSY
Follow-up to the URDF assembly support, along four lines.

**Links are parts.** A URDF link becomes exactly one part of the package, named
'<assembly>/<link>' and expressed in the link's own frame. The "internal" marker
is gone: these are ordinary parts, so 'pc inspect robot/forearm' and
'pc export -t step robot/wrist' work on them. They are still declared by the
URDF rather than by 'partcad.yaml', so 'Project.get_part' builds the assembly
that owns such a name before reporting it missing. A link with several visuals
is combined into one shape rather than becoming a sub-assembly, which is what
puts the part's origin on the link's and lets a joint attach to it without a
correction.

**Collision geometry wins.** A link that states both is built from its collision
shape - what a simulator resolves contact against. 'ignoreCollision', either
true or a list of link names, selects the visual shape instead.

**Nothing is silently dropped.** Parts gain an opaque 'physics:' section and
interfaces gain 'motion:' and 'physics:', each keyed by the format the contents
came from. A URDF import fills them - mass, inertia, materials, the geometry it
did not build from, '<gazebo>' blocks; joint type, axis, limits, dynamics - and
the URDF export puts them back, so a stated mass is no longer replaced by a
computed one.

**'pc convert assembly'.** To URDF it writes the '.urdf' and its meshes. To ASSY
it writes an stl part per link, an interface pair per joint, and an '.assy' that
places its parts with 'connect:'. A URDF joint becomes a "socket" interface the
parent implements at the joint origin and a "plug" the child implements at its
own, mating; joints that say the same thing share one pair. The movable ones
also get an interface parameter, so 'toParams: {angle: 90}' in the generated
ASSY poses the joint in the URDF sense. 'pc adhoc convert' refuses both formats,
since neither means anything without a package.

Two long-standing gaps surfaced from generating interfaces programmatically:
'ports: {name:}' and 'implements: {iface:}' with no value are both legal per the
schema and both crashed. The schema also did not allow 'type: turn' on a custom
interface parameter, which the documentation has always shown.

docs/source/simulation.rst records the joint-to-interface mapping, why the half
turn lands on the plug, and what the proposal still needs.

Co-Authored-By: Claude Opus 5 <noreply@anthropic.com>
Claude-Session: https://claude.ai/code/session_01TyEL5ea3RRyJ8QhD2WwcUV

File: examples/produce_assembly_urdf/robot.urdf (robot description, URDF)
Before this commit: robot partcad_urdf_example, 4 links, 3 joints
Links:
- link base_link: geometry collision box size=0.13 0.13 0.02; visual box size=0.12 0.12 0.02
- link wrist: geometry collision mesh filename=package://produce_part_stl/cube.stl scale=0.001 0.001 0.001; visual mesh filename=package://produce_part_stl/cube.stl scale=0.001 0.001 0.001

Commit message: Write URDF joints from the body rule, and read and convert a URDF as the mechanism it is
Step 11 of the simulation design record (section 8.8b).

The URDF exporter writes a link per rigid body and a joint per pair of
bodies, from kinematics.bodies() and classify() and nothing of its own:
revolute, continuous, prismatic, planar (its axis the normal) and floating
natively; a cylindrical, universal, ball or screw joint and a chain as one
single-axis joint per freedom through dummy links '<joint>_link<n>' of a
small mass and inertia, a screw's move a <mimic> of its turn by the lead.
The child link's frame is the joint's moving frame, so <axis> is the
freedom's axis verbatim and every part sits in its link at the joint's
tail; each part of a body is a <visual>/<collision> of its own, named after
it, and the body's combined physics is the <inertial>. A free root is the
root link where the tree put it; a body fixed to the world hangs off
'world' by a fixed joint, and a scene's free bodies by floating ones.
Metres and radians at the boundary only. What URDF cannot state is
reported: the starting value (written at zero), dummy links, the effort
and velocity URDF requires where a joint states none (the export's
'effort' and 'velocity' parameters), an open bound. Everything up to
urdf_parser_py is a plain-data Planner the tests move through
configurations, one test per row of the classification table.

The URDF reader states each link node's joint in the envelope form - the
parent's shape offset undone, each joint origin and the freedoms it keeps,
the link's shape offset - and a link on a fixed joint the link it is
attached to. AssemblyFactoryImported builds AssemblyChild.joint from it
with the new Joint.from_envelope, knowing no format, so a 'type: urdf'
assembly is a mechanism without converting it, and 'pc info -a' lists its
joints. A joint with no <axis> turns about URDF's default X (the gap #766
found), joints through a link with no geometry are one joint, and a
mimic is restated in PartCAD's units on both sides. Movable joints are
no longer counted as dropped.

The converter writes the explicit 'motion: {dof: [...]}' form, one
parameter per freedom from the reader's own list, and moves the half turn
from the plug to the socket's port: the contact frame is the URDF joint
frame, every parameter's dir is the URDF axis verbatim, 'connect: {joint:}'
keeps the URDF's name, and exporting a converted URDF gives its frames and
axes back. Interfaces are still deduplicated on the reader's record.

Two additions to the helper, both needed by the round trip: a rigid
connection now says what it is attached to (shape_envelope.KEY_ATTACHED,
stamped by Assembly._place in assemblies), and bodies() welds such a child
into its target's body - a forearm fixed to a turning shoulder turned
with the base before; and a joint naming no sibling is to the container.
The payload changed, so the cache format is 11.

The example's wrist is a continuous joint now, so the example shows a
turning joint, a fixed one under it and a second movable one; its README
is re-rendered and its drawing is unchanged.

Co-Authored-By: Claude Opus 5.5 <noreply@anthropic.com>
Claude-Session: https://claude.ai/code/session_01W75xcC24VB11oxbGUr1N1T

File: examples/produce_assembly_urdf/robot.urdf (robot description, URDF)
Before this commit: robot partcad_urdf_example, 4 links, 3 joints
Joints:
- joint wrist: axis (none) -> 0 0 1; type fixed -> continuous
